Commit message: Updated p2os repo

File: p2os/p2os_urdf/defs/pioneer3dx.urdf.xacro (robot description, xacro)
@@ -17,5 +17,5 @@
 				 izz="1"/>
 		</inertial>
-		<visual name="base_visual">
+		<visual>
 			<origin xyz="-0.045 0 0.148" rpy="0 0 0"/>
 			<geometry name="pioneer_geom">
@@ -33,6 +33,11 @@
 		</collision>
 	</link>
-<!-- Top -->
-	<link name="top_plate">
+    <joint name="base_top_joint" type="fixed">
+		<origin xyz="-0.045 0 0.234" rpy="0 0 0"/>
+		<axis xzy="0 0 1"/>
+		<parent link="base_link"/>
+		<child link="top_plate"/>
+	</joint>
+	<link name="base_top">
 		<inertial>
 			<mass value="0"/>
@@ -42,5 +47,5 @@
  				izz="1"/>
 		</inertial>
-		<visual name="base_visual">
+		<visual>
 			<origin xyz="0 0 0" rpy="0 0 0"/>
 			<geometry name="pioneer_geom">
@@ -58,9 +63,4 @@
 		</collision>
 	</link>
-	<joint name="base_top_joint" type="fixed">
-		<origin xyz="-0.045 0 0.234" rpy="0 0 0"/>
-		<parent link="base_link"/>
-		<child link="top_plate"/>
-	</joint>
 <!-- Swivel -->
 	<link name="swivel">
@@ -188,4 +188,9 @@
 		<child link="front_sonar"/>
 	</joint>
+	<joint name="base_back_joint" type="fixed">
+		<origin xyz="0.109 0 0.209" rpy="0 0 0"/>
+		<parent link="base_link"/>
+		<child link="back_sonar"/>
+	</joint>
 	<link name="back_sonar">
 		<inertial>
@@ -211,9 +216,8 @@
 		</collision>
 	</link>
-	<joint name="base_back_joint" type="fixed">
-		<origin xyz="0.109 0 0.209" rpy="0 0 0"/>
-		<parent link="base_link"/>
-		<child link="back_sonar"/>
-	</joint>
+	<create>
+	<back_sonar parent="base_link"/>
+  	<top_plate  parent="base_link"/>
+  	</create>
 <gazebo>
 	<controller:differential_position2d name="controller1">

File: p2os/p2os_urdf/defs/pioneer3dx.xacro (robot description, xacro)
@@ -8,12 +8,4 @@
 <!-- Chassis -->
 	<link name="base_link">
-		<inertial>
-			<mass value="3.5"/>
-			<!--<origin xyz="-0.025 0 -0.223"/>-->
-			<origin xyz="-0.05 0 0"/>
-			<inertia ixx="1" ixy="0" ixz="0"
-				 iyy="1" iyz="0"
-				 izz="1"/>
-		</inertial>
 		<visual name="base_visual">
 			<origin xyz="-0.045 0 0.148" rpy="0 0 0"/>
@@ -25,24 +17,13 @@
 			</material>
 		</visual>
-		<collision>
-			<origin xyz="-0.045 0 0.145" rpy="0 0 0"/>
-				<geometry>
-					<box size="0.35 0.25 0.14"/>
-				</geometry>
-		</collision>
-	</link>
-	<gazebo reference="base_link">
-		<material value="Gazebo/Red"/>
-	</gazebo>
+	</link>
 <!-- Top -->
+	<joint name="base_top_joint" type="fixed">
+		<origin xyz="-0.045 0 0.234" rpy="0 0 0"/>
+		<parent link="base_link"/>
+		<child link="top_plate"/>
+	</joint>
 	<link name="top_plate">
-		<inertial>
-			<mass value="0.01"/>
-			<origin xyz="0 0 0"/>
-			<inertia ixx="1" ixy="0" ixz="0"
-				 iyy="1" iyz="0"
- 				izz="1"/>
-		</inertial>
-		<visual name="base_visual">
+		<visual>
 			<origin xyz="0 0 0" rpy="0 0 0"/>
 			<geometry name="top_geom">
@@ -53,20 +34,14 @@
 			</material>
 		</visual>
-		<collision>
-			<origin xyz="0.0 0 0" rpy="0 0 0"/>
-			<geometry name="pioneer_geom">
-				<box size="0.45 0.38 0.01"/>
-			</geometry>
-		</collision>
-	</link>
-	<gazebo reference="top_plate">
-		<material value="Gazebo/Black"/>
-	</gazebo>
-	<joint name="base_top_joint" type="fixed">
-		<origin xyz="-0.045 0 0.234" rpy="0 0 0"/>
-		<parent link="base_link"/>
-		<child link="top_plate"/>
-	</joint>
+	</link>
 <!-- Swivel -->
+	<joint name="base_swivel_joint" type="continuous">
+		<origin xyz="-0.185 0 0.055" rpy="0 0 0"/>
+		<anchor xyz="0 0 0"/>
+    	<limit effort="100" velocity="100" k_velocity="0" />
+    	<joint_properties damping="0.0" friction="0.0" />
+		<parent link="base_link"/>
+		<child link="swivel"/>
+	</joint>
 	<link name="swivel">
 		<inertial>
@@ -92,16 +67,4 @@
 	</collision>
 	</link>
-	<gazebo reference="swivel">
-		<material value="Gazebo/Grey"/>
-	</gazebo>
- 	<joint name="base_swivel_joint" type="continuous">
-		<origin xyz="-0.185 0 0.055" rpy="0 0 0"/>
-		<axis xyz="0 0 1"/>
-		<anchor xyz="0 0 0"/>
-    <limit effort="100" velocity="100" k_velocity="0" />
-    <joint_properties damping="0.0" friction="0.0" />
-		<parent link="base_link"/>
-		<child link="swivel"/>
-	</joint>
 <!-- Center Wheel + Hubcap -->
 	<link name="center_hubcap">
@@ -169,13 +132,70 @@
 		<child link="center_hubcap"/>
 	</joint>
-	<gazebo reference="center_wheel">
-		<material value="Gazebo/Black"/>
-    <elem key="mu1" value="10.0" />
-    <elem key="mu2" value="10.0" />
-    <elem key="kp"  value="1000000.0" />
-    <elem key="kd"  value="1.0" />
-	</gazebo>
-<xacro:p3dx_wheel suffix="left" parent="base_link" reflect="1"/>
-<xacro:p3dx_wheel suffix="right" parent="base_link" reflect="-1"/>
+	<link name="left_hub">
+		<visual>
+			<origin xyz="0 0 0" rpy="0 0 0"/>
+			<geometry>
+				<mesh filename="package://p2os_urdf/meshes/p3dx_meshes/left_hubcap.stl"/>
+			</geometry>
+			<material name="HubcapYellow">
+				<color rgba="1.0 0.811 0.151 1.0"/>
+			</material>
+		</visual>
+	</link>
+	<joint name="left_hub_joint" type="fixed">
+		<origin xyz="0 0.15 0.08" rpy="0 0 0"/>
+		<parent link="base_link"/>
+		<child link="left_hub"/>
+		<axis xyz="0 1 0"/>
+	</joint>
+	<link name="left_wheel_joint">
+		<visual>
+			<origin xyz="0 0 0" rpy="0 0 0"/>
+			<geometry>
+				<mesh filename="package://p2os_urdf/meshes/p3dx_meshes/left_wheel.stl"/>
+			</geometry>
+			<material name="WheelBlack">
+				<color rgba="0.117 0.117 0.117 1"/>
+			</material>
+		</visual>
+	</link>
+	<joint name="left_wheel_joint" type="fixed">
+		<origin xyz="0 0 0" rpy="0 0 0"/>
+		<parent link="left_hub"/>
+		<child link="left_wheel_joint"/>
+	</joint>
+	<link name="right_hub">
+		<visual>
+			<origin xyz="0 0 0" rpy="0 0 0"/>
+			<geometry>
+				<mesh filename="package://p2os_urdf/meshes/p3dx_meshes/right_hubcap.stl"/>
+			</geometry>
+			<material name="HubcapYellow">
+				<color rgba="1.0 0.811 0.151 1.0"/>
+			</material>
+		</visual>
+	</link>
+	<joint name="right_hub_joint" type="fixed">
+		<origin xyz="0 -0.15 0.08" rpy="0 0 0"/>
+		<parent link="base_link"/>
+		<child link="right_hub"/>
+		<axis xyz="0 1 0"/>
+	</joint>
+	<link name="right_wheel_joint">
+		<visual>
+			<origin xyz="0 0 0" rpy="0 0 0"/>
+			<geometry>
+				<mesh filename="package://p2os_urdf/meshes/p3dx_meshes/right_wheel.stl"/>
+			</geometry>
+			<material name="WheelBlack">
+				<color rgba="0.117 0.117 0.117 1"/>
+			</material>
+		</visual>
+	</link>
+	<joint name="right_wheel_joint" type="fixed">
+		<origin xyz="0 0 0" rpy="0 0 0"/>
+		<parent link="right_hub"/>
+		<child link="right_wheel_joint"/>
+	</joint>
 <!-- Front + Back Sonar -->
 	<link name="front_sonar">
