Commit message: updated p2os code

File: p2os/p2os_urdf/defs/pioneer3dx.xacro (robot description, xacro)
@@ -18,4 +18,7 @@
 		</visual>
 	</link>
+	<gazebo reference="base_link">
+		<material value="Gazebo/Red"/>
+	</gazebo>
 <!-- Top -->
 	<joint name="base_top_joint" type="fixed">
@@ -26,4 +29,11 @@
 	<link name="top_plate">
 		<visual>
+			<inertial>
+				<mass value="0.01"/>
+				<origin xyz="0 0 0"/>
+				<inertia ixx="1" ixy="0" ixz="0"
+					 iyy="1" iyz="0"
+	 				izz="1"/>
+			</inertial>
 			<origin xyz="0 0 0" rpy="0 0 0"/>
 			<geometry name="top_geom">
@@ -35,4 +45,7 @@
 		</visual>
 	</link>
+	<gazebo reference="top_plate">
+		<material value="Gazebo/Black"/>
+	</gazebo>
 <!-- Swivel -->
 	<joint name="base_swivel_joint" type="continuous">
@@ -67,4 +80,7 @@
 	</collision>
 	</link>
+	<gazebo reference="swivel">
+		<material value="Gazebo/Grey"/>
+	</gazebo>
 <!-- Center Wheel + Hubcap -->
 	<link name="center_hubcap">
@@ -262,6 +278,8 @@
 	</joint>
   <gazebo>
-    <controller:differential_position2d name="controller1">
+    <controller:diffdrive_plugin name="differential_drive_controller" plugin="libdiffdrive_plugin.so">
+      <alwaysOn>true</alwaysOn>
       <update>100</update>
+      <updateRate>100.0</updateRate>
       <leftJoint>base_right_wheel_joint</leftJoint>
       <rightJoint>base_left_wheel_joint</rightJoint>
@@ -270,5 +288,7 @@
       <torque>5</torque>
       <interface:position name="position_iface_0"/>
-    </controller:differential_position2d>
+      <robotNamespace>/</robotNamespace>
+      <topicName>cmd_vel</topicName>
+    </controller:diffdrive_plugin>
     <controller:gazebo_ros_p3d name="p3d_base_controller" plugin="libgazebo_ros_p3d.so">
       <alwaysOn>true</alwaysOn>
@@ -282,7 +302,4 @@
       <interface:position name="p3d_base_position"/>
     </controller:gazebo_ros_p3d>
-    <!-- this publishes empty joint_states due to no transmission, but
-         triggering robot_state_puublisher to publish tf between fixed joints in erratic,
-         (e.g. base_laser_link for the base_scan frame) -->
     <controller:gazebo_ros_controller_manager name="gazebo_ros_controller_manager" plugin="libgazebo_ros_controller_manager.so">
       <alwaysOn>true</alwaysOn>
